File: Tarea 3/Proyecto board puerta/Board_Micro.kicad_sch (KiCad schematic)
At the start: 7 parts, among them U3 ESP32-DEVKITC

Commit message: Actualizando proyecto kiCAD
Parts:
- added C5, C6, C7, C8: 100nF_0603_16V, 4ms_Capacitor:C_0603, symbol PCM_4ms_Capacitor:100nF_0603_16V
- added Q3, Q4: PNP, Package_TO_SOT_SMD:SOT-223-3_TabPin2, symbol Transistor_BJT:PZT2222A
- added R10, R3, R4, R6, R7, R9: 1k, Resistor_SMD:R_0402_1005Metric, symbol Device:R_Small_US
Connections:
- net LSA is gone; now on net LSA_M: C3.1, R17.1
- net LSC is gone; now on net LSC_M: C2.1, R2.2
- net GND: now also U3.2 (GND), C5.2, C6.2, C7.2, C8.2, Q3.3 (E), Q4.3 (E)
- net VDD: now also U3.1 (3V3), R3.2, R4.2, R6.2, R7.2
- net KEYC_M: now reaches U3.10 (D19)
- net KEYC_M: now also C5.1, R6.1
- net KEYA_M: now reaches U3.11 (D21)
- net KEYA_M: now also C6.1, R7.1
- net Bzzr_from_Micro: now reaches U3.19 (D34)
- net Bzzr_from_Micro: now also R10.1
- net Light_from_Micro: now reaches U3.21 (D32)
- net Light_from_Micro: now also R9.1
- net LSA_M: now reaches U3.4 (D2)
- net LSC_M: now reaches U3.5 (D4)
- net FTC_M: now reaches U3.8 (D5)
- net FTC_M: now also C8.1, R4.1
- net PP_M: now reaches U3.9 (D18)
- net PP_M: now also C7.1, R3.1
- new net: Q4.1 (B), R10.2
- new net: Q3.1 (B), R9.2
- new net to_Buzzer: Q4.2 (C)
- new net to_Light: Q3.2 (C)
