File: Tarea 3/Proyecto board puerta/Proyecto board puerta.kicad_sch (KiCad schematic)
At the start: 29 parts, among them J1 LIMIT SWITCHES, J2 KEY, J3 PP, J4 Light, J5 MOTOR, J6 VIn, J7 Fotocelda, K1 Relay 2, K2 Relay 1, Q1 PNP, Q2 PNP, Q3 PNP, Q4 PNP

Commit message: Actualizando proyecto KiCAD
Parts:
- removed J1: LIMIT SWITCHES, TerminalBlock:TerminalBlock_bornier-3_P5.08mm, symbol Connector:Screw_Terminal_01x03
- removed J6: VIn, TerminalBlock:TerminalBlock_bornier-2_P5.08mm, symbol Connector:Screw_Terminal_01x02
- removed R1, R2: 1k, Resistor_SMD:R_0402_1005Metric, symbol Device:R_Small_US
- added D3: ESD9B3.3ST5G, Diode_SMD:D_SOD-923, symbol Diode:ESD9B3.3ST5G
- added J10: FTC, TerminalBlock:TerminalBlock_bornier-3_P5.08mm, symbol Connector:Screw_Terminal_01x03
- added J11: idk1, TerminalBlock:TerminalBlock_bornier-3_P5.08mm, symbol Connector:Screw_Terminal_01x03
- added J12: Screw_Terminal_01x02, symbol Connector:Screw_Terminal_01x02
- added J8: Limit Switch, TerminalBlock:TerminalBlock_bornier-3_P5.08mm, symbol Connector:Screw_Terminal_01x03
- added J9: idk2, TerminalBlock:TerminalBlock_bornier-3_P5.08mm, symbol Connector:Screw_Terminal_01x03
- added R13, R14, R15, R16: 1k, Resistor_SMD:R_0402_1005Metric, symbol Device:R_Small_US
- added SW1: SW_DIP_x04, Button_Switch_SMD:SW_DIP_SPSTx04_Slide_9.78x12.34mm_W8.61mm_P2.54mm, symbol Switch:SW_DIP_x04
- added SW2: Dip Switch, symbol Switch:SW_DIP_x04
- added SW3: Btn_Reset, symbol Switch:SW_MEC_5E
- added U1: ESP32-DEVKITC, LIBRERIA PERSONAL:MODULE_ESP32-DEVKITC, symbol ESP32-DEVKITC:ESP32-DEVKITC
Connections:
- net +3.3V: now also R13.1, R14.1, R15.1, R16.1, U1.1 (3V3), U1.10 (D19), U1.9 (D18)
- net +5V: now also U1.30 (VIN)
- net FTC: now also U1.8 (D5)
- net GND: now also D3.1 (A1), J12.2 (Pin_2), J8.2 (Pin_2), SW1.5, SW1.6, SW1.7, SW1.8, SW2.1, SW2.2, SW2.3, SW2.4, SW3.1, SW3.2, U1.2 (GND)
- net MA: now also U1.24 (D26)
- net MC: now also U1.23 (D25)
- net PP: now also U1.11 (D21)
- new net: R13.2, SW1.1, U1.28 (D13)
- new net: R16.2, SW1.4, U1.25 (D27)
- new net: R15.2, SW1.3, U1.26 (D14)
- new net: R14.2, SW1.2, U1.27 (D12)
- new net BUZZER: U1.19 (D34)
- new net Board_Micro/DIP1: SW2.8
- new net Board_Micro/DIP2: SW2.7
- new net Board_Micro/DIP3: SW2.6
- new net Board_Micro/DIP4: SW2.5
- new net Board_Micro/LSA: J8.1 (Pin_1)
- new net Board_Micro/LSC: J8.3 (Pin_3)
- new net Board_Micro/MOTOR_LEFT: J11.3 (Pin_3)
- new net Board_Micro/MOTOR_RIGHT: J11.1 (Pin_1)
- new net Board_Micro/RST: D3.2 (A2), SW3.3 (K), SW3.4 (A)
- new net LAMP: U1.21 (D32)
- new net LSA: U1.5 (D4)
- new net LSC: U1.4 (D2)
- new net VDD: J12.1 (Pin_1)
Other:
- added sheet Board_Micro (Board_Micro.kicad_sch)
- moved on the sheet: BZ1

Commit message: Actualizando proyecto kiCAD
Parts:
- removed BZ1: Buzzer, Buzzer_Beeper:Buzzer_CUI_CPT-9019S-SMT, symbol Device:Buzzer
- removed C1: 22u, Capacitor_SMD:C_0402_1005Metric, symbol Device:C_Small
- removed D1: CLOSED LED, LED_SMD:LED_0402_1005Metric, symbol Device:LED
- removed D2: OPEN LED, LED_SMD:LED_0402_1005Metric, symbol Device:LED
- removed J2: KEY, TerminalBlock:TerminalBlock_bornier-3_P5.08mm, symbol Connector:Screw_Terminal_01x03
- removed J3: PP, TerminalBlock:TerminalBlock_bornier-2_P5.08mm, symbol Connector:Screw_Terminal_01x02
- removed J4: Light, TerminalBlock:TerminalBlock_bornier-2_P5.08mm, symbol Connector:Screw_Terminal_01x02
- removed J7: Fotocelda, TerminalBlock:TerminalBlock_bornier-3_P5.08mm, symbol Connector:Screw_Terminal_01x03
- removed J9: idk2, TerminalBlock:TerminalBlock_bornier-3_P5.08mm, symbol Connector:Screw_Terminal_01x03
- removed K1: Relay 2, Relay_THT:Relay_SPDT_Finder_36.11, symbol Relay:FINDER-36.11
- removed K2: Relay 1, Relay_THT:Relay_SPDT_Finder_36.11, symbol Relay:FINDER-36.11
- removed Q1, Q2, Q3, Q4: PNP, Package_TO_SOT_SMD:SOT-223-3_TabPin2, symbol Transistor_BJT:PZT2222A
- removed R10, R11, R13, R14, R15, R16, R3, R4, R5, R6, R7, R8: 1k, Resistor_SMD:R_0402_1005Metric, symbol Device:R_Small_US
- removed R12, R9: 220, Resistor_SMD:R_0402_1005Metric, symbol Device:R_Small_US
- removed SW1: SW_DIP_x04, Button_Switch_SMD:SW_DIP_SPSTx04_Slide_9.78x12.34mm_W8.61mm_P2.54mm, symbol Switch:SW_DIP_x04
- removed U1: ESP32-DEVKITC, LIBRERIA PERSONAL:MODULE_ESP32-DEVKITC, symbol ESP32-DEVKITC:ESP32-DEVKITC
- added J1: PP, TerminalBlock:TerminalBlock_bornier-2_P5.08mm, symbol Connector:Screw_Terminal_01x02
- added J4: KEY, TerminalBlock:TerminalBlock_bornier-3_P5.08mm, symbol Connector:Screw_Terminal_01x03
- added J6: Buzzer, TerminalBlock:TerminalBlock_bornier-2_P5.08mm, symbol Connector:Screw_Terminal_01x02
- J11: value idk1 -> Motor
- J5: value MOTOR -> Light
Connections:
- net M1 is gone; now on net VDD: J5.2 (Pin_2)
- net Board_Micro/+_CON_FTC: now also J10.1 (Pin_1)
- net Board_Micro/-_CON_FTC: now also J10.3 (Pin_3)
- net Board_Micro/CON_IN_FTC: now also J10.2 (Pin_2)
- net GND: now also J1.2 (Pin_2), J4.3 (Pin_3)
- net VDD: now also J6.2 (Pin_2)
- net M2 renamed Board_Micro/to_Light
- new net Board_Micro/KeyA: J4.1 (Pin_1)
- new net Board_Micro/KeyC: J4.2 (Pin_2)
- new net Board_Micro/PP: J1.1 (Pin_1)
- new net Board_Micro/to_Buzzer: J6.1 (Pin_1)
Other:
- sheet Board_Micro ports: added KeyA, KeyC, PP, to_Buzzer, to_Light; removed none
