File: Tarea 3/Proyecto board puerta/motor_driver_rly.kicad_sch (KiCad schematic)
At the start: 10 parts, among them K3 Relay 2, K4 Relay 1, Q6 PNP, Q7 PNP

Commit message: Actualizando proyecto kiCAD
Connections:
- net +5V renamed VDD
Changed lines of the file:
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@@
 	(wire
 		(pts
-			(xy 59.69 96.52) (xy 59.69 97.79)
+			(xy 59.69 96.52) (xy 59.69 99.06)
 		)
 		(stroke
@@
 	(wire
 		(pts
-			(xy 144.78 54.61) (xy 149.86 54.61)
+			(xy 80.01 73.66) (xy 80.01 71.12)
 		)
 		(stroke
@@
 	(wire
 		(pts
-			(xy 80.01 71.12) (xy 83.82 71.12)
-		)
-		(stroke
-			(width 0)
-			(type default)
-		)
-	)
-	(wire
-		(pts
 			(xy 59.69 93.98) (xy 59.69 96.52)
 		)
@@
 		(pts
 			(xy 133.35 54.61) (xy 132.08 54.61)
+		)
+		(stroke
+			(width 0)
+			(type default)
+		)
+	)
+	(wire
+		(pts
+			(xy 144.78 57.15) (xy 144.78 54.61)
 		)
 		(stroke
@@
 	(hierarchical_label "MOTOR1"
 		(shape input)
-		(at 149.86 54.61 0)
+		(at 144.78 57.15 270)
 		(effects
 			(font
 				(size 1.27 1.27)
 			)
-			(justify left)
+			(justify right)
 		)
 	)
@@
 	(hierarchical_label "MOTOR2"
 		(shape input)
-		(at 83.82 71.12 0)
+		(at 80.01 73.66 270)
 		(effects
 			(font
 				(size 1.27 1.27)
 			)
-			(justify left)
+			(justify right)
 		)
 	)
 	(symbol
-		(lib_id "power:+5V")
-		(at 59.69 97.79 180)
+		(lib_id "power:VDD")
+		(at 124.46 81.28 180)
 		(unit 1)
 		(exclude_from_sim no)
@@
 		(dnp no)
 		(fields_autoplaced yes)
-		(property "Reference" "#PWR3"
-			(at 59.69 93.98 0)
-			(effects
-				(font
-					(size 1.27 1.27)
-				)
-				(hide yes)
-			)
-		)
-		(property "Value" "+5V"
-			(at 59.69 102.87 0)
+		(property "Reference" "#PWR16"
+			(at 124.46 77.47 0)
+			(effects
+				(font
+					(size 1.27 1.27)
+				)
+				(hide yes)
+			)
+		)
+		(property "Value" "VDD"
+			(at 124.46 86.36 0)
 			(effects
 				(font
@@
 		)
 		(property "Footprint" ""
-			(at 59.69 97.79 0)
+			(at 124.46 81.28 0)
 			(effects
 				(font
@@
 		)
 		(property "Datasheet" ""
-			(at 59.69 97.79 0)
-			(effects
-				(font
-					(size 1.27 1.27)
-				)
-				(hide yes)
-			)
-		)
-		(property "Description" "Power symbol creates a global label with name \"+5V\""
-			(at 59.69 97.79 0)
+			(at 124.46 81.28 0)
+			(effects
+				(font
+					(size 1.27 1.27)
+				)
+				(hide yes)
+			)
+		)
+		(property "Description" "Power symbol creates a global label with name \"VDD\""
+			(at 124.46 81.28 0)
 			(effects
 				(font
@@
 			(project "Proyecto board puerta"
 				(path "/10750c3a-d383-45d6-b98c-cd879b600e84/470d22ce-1fe2-4179-8d6b-55797b69dbf4/842155f9-e599-44a4-a3e5-6e181bbdea1b"
-					(reference "#PWR3")
+					(reference "#PWR16")
 					(unit 1)
 				)
@@
 	)
 	(symbol
-		(lib_id "power:+5V")
-		(at 124.46 81.28 180)
+		(lib_id "power:VDD")
+		(at 59.69 99.06 180)
 		(unit 1)
 		(exclude_from_sim no)
@@
 		(dnp no)
 		(fields_autoplaced yes)
-		(property "Reference" "#PWR47"
-			(at 124.46 77.47 0)
-			(effects
-				(font
-					(size 1.27 1.27)
-				)
-				(hide yes)
-			)
-		)
-		(property "Value" "+5V"
-			(at 124.46 86.36 0)
+		(property "Reference" "#PWR15"
+			(at 59.69 95.25 0)
+			(effects
+				(font
+					(size 1.27 1.27)
+				)
+				(hide yes)
+			)
+		)
+		(property "Value" "VDD"
+			(at 59.69 104.14 0)
 			(effects
 				(font
@@
 		)
 		(property "Footprint" ""
-			(at 124.46 81.28 0)
+			(at 59.69 99.06 0)
 			(effects
 				(font
@@
 		)
 		(property "Datasheet" ""
-			(at 124.46 81.28 0)
-			(effects
-				(font
-					(size 1.27 1.27)
-				)
-				(hide yes)
-			)
-		)
-		(property "Description" "Power symbol creates a global label with name \"+5V\""
-			(at 124.46 81.28 0)
+			(at 59.69 99.06 0)
+			(effects
+				(font
+					(size 1.27 1.27)
+				)
+				(hide yes)
+			)
+		)
+		(property "Description" "Power symbol creates a global label with name \"VDD\""
+			(at 59.69 99.06 0)
 			(effects
 				(font
@@
 			(project "Proyecto board puerta"
 				(path "/10750c3a-d383-45d6-b98c-cd879b600e84/470d22ce-1fe2-4179-8d6b-55797b69dbf4/842155f9-e599-44a4-a3e5-6e181bbdea1b"
-					(reference "#PWR47")
+					(reference "#PWR15")
 					(unit 1)
 				)
