File: Tarea 3/Proyecto board puerta/Proyecto board puerta.kicad_pcb (KiCad board)
At the start: 2 copper layers, 39 parts, among them J10 idk3, J11 idk1, J2 KEY, J3 PP, J4 Light, J5 MOTOR, J6 VIn, J7 Fotocelda, J8 idk1, J9 idk2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

Commit message: Tarea 5
Parts:
- added D3: ESD9B3.3ST5G, Diode_SMD:D_SOD-923, F.Cu at (75.0, 40.5)
- added D4: CLOSED LED, LED_SMD:LED_0402_1005Metric, F.Cu at (40.7, 51.8)
- added D5: OPEN LED, LED_SMD:LED_0402_1005Metric, F.Cu at (40.7, 53.8)
- added J1: PP, TerminalBlock:TerminalBlock_bornier-2_P5.08mm, F.Cu at (65.3, 35.0)
- added J4: KEY, TerminalBlock:TerminalBlock_bornier-3_P5.08mm, F.Cu at (76.8, 35.0)
- added J5: Light, TerminalBlock:TerminalBlock_bornier-2_P5.08mm, F.Cu at (65.3, 44.0)
- added J6: Buzzer, TerminalBlock:TerminalBlock_bornier-2_P5.08mm, F.Cu at (65.3, 53.1)
- added K3: Relay 2, Relay_THT:Relay_SPDT_Finder_36.11, F.Cu at (28.8, 34.5)
- added K4: Relay 1, Relay_THT:Relay_SPDT_Finder_36.11, F.Cu at (45.7, 34.5)
- added Q3: PNP, Package_TO_SOT_SMD:SOT-223-3_TabPin2, F.Cu at (67.0, 63.8)
- added Q4: PNP, Package_TO_SOT_SMD:SOT-223-3_TabPin2, F.Cu at (67.0, 72.2)
- added Q6: PNP, Package_TO_SOT_SMD:SOT-223-3_TabPin2, F.Cu at (31.2, 55.0)
- added Q7: PNP, Package_TO_SOT_SMD:SOT-223-3_TabPin2, F.Cu at (31.2, 63.4)
- added R10: 1k, Resistor_SMD:R_0402_1005Metric, F.Cu at (73.3, 70.6)
- added R18: 1k, Resistor_SMD:R_0402_1005Metric, F.Cu at (37.6, 51.8)
- added R19: 220, Resistor_SMD:R_0402_1005Metric, F.Cu at (37.6, 53.8)
- added R20: 1k, Resistor_SMD:R_0402_1005Metric, F.Cu at (37.6, 55.8)
- added R21: 220, Resistor_SMD:R_0402_1005Metric, F.Cu at (37.6, 57.8)
- added R3: 1k, Resistor_SMD:R_0402_1005Metric, F.Cu at (73.3, 60.6)
- added R4: 1k, Resistor_SMD:R_0402_1005Metric, F.Cu at (73.3, 62.6)
- added R6: 1k, Resistor_SMD:R_0402_1005Metric, F.Cu at (73.3, 64.6)
- added R7: 1k, Resistor_SMD:R_0402_1005Metric, F.Cu at (73.3, 66.6)
- added R9: 1k, Resistor_SMD:R_0402_1005Metric, F.Cu at (73.3, 68.6)
- J10: value idk3 -> FTC
- J11: value idk1 -> Motor
- J8: value idk1 -> Limit Switch
Connections:
- net /Board_Micro/LSA renamed LSA_M
- net /Board_Micro/LSC renamed LSC_M
- J10 pad 1: unconnected-(J10-Pin_1-Pad1) -> VDD
- J10 pad 2: unconnected-(J10-Pin_2-Pad2) -> FTC_M
- J10 pad 3: unconnected-(J10-Pin_3-Pad3) -> GND
- J11 pad 1: unconnected-(J11-Pin_1-Pad1) -> /Board_Micro/MOTOR_RIGHT
- J11 pad 3: unconnected-(J11-Pin_3-Pad3) -> /Board_Micro/MOTOR_LEFT
